File: ref_ver_1.kicad_sch (KiCad schematic)
At the start: 21 parts, among them J1 Conn_01x03_Pin, J2 Conn_01x03_Pin, J3 Conn_01x03_Pin, J4 Conn_01x04_Pin, U1 LM399, U2 LTC2057IS8-TRPBF, U3 SHT4x

Commit message: updated to new revision
Parts:
- added C7: 100n, Capacitor_SMD:C_0603_1608Metric_Pad1.08x0.95mm_HandSolder, symbol Device:C
- added C8: 10n, Capacitor_SMD:C_0603_1608Metric_Pad1.08x0.95mm_HandSolder, symbol Device:C
Connections:
- net GND: now also C7.2
- net IN-: now also C8.1
- net OUT: no longer R1.3, R3.2
- net VCC: now also C7.1
- net at C5.1, J2.3 (Pin_3), R5.2: now also R1.3, R3.2, C8.2
Other:
- moved on the sheet: C1, C2, D1, J1, R5
